Commit message: Minor adjustments in camera and laser sensor parameters to improve sensor feed

File: robot_19/urdf/robot_19.urdf (robot description, URDF)
Before this commit: robot robot_19, 5 links, 4 joints
Links:
- added link camera_link, mass 0.5; collision box size=0.01 0.01 0.3; visual box size=0.01 0.01 0.3
- added link laser_link, mass 0.5; collision box size=0.01 0.01 0.05; visual box size=0.01 0.01 0.05
Joints:
- added joint joint_sensor_camera: type fixed, parent base_link, child camera_link, origin xyz=-0.15 0 0.255 rpy=0 0 0
- added joint joint_sensor_laser: type fixed, parent base_link, child laser_link, origin xyz=0.15 0 0.105 rpy=0 0 0
- joint Slider_joint: limit lower=-3 upper=-0.5 effort=1000 velocity=0.5 -> lower=-3 upper=-0.1 effort=1000 velocity=0.5
