Commit message: Added laser link and sensor to the new box robot design

File: box_robot11/urdf/box_robot11.urdf (robot description, URDF)
Before this commit: robot box_robot11, 6 links, 5 joints
Links:
- added link laser_link, mass 0.5; collision box size=0.01 0.01 0.05; visual box size=0.05 0.05 0.05
Joints:
- added joint joint_sensor_laser: type fixed, parent base_link, child laser_link, origin xyz=0.225 0 0.105 rpy=0 0 0

Commit message: Added camera link and sensor to the new box robot design

File: box_robot11/urdf/box_robot11.urdf (robot description, URDF)
Before this commit: robot box_robot11, 7 links, 6 joints
Links:
- added link camera_link, mass 0.5; collision box size=0.01 0.01 0.25; visual box size=0.05 0.05 0.25
Joints:
- added joint joint_sensor_camera: type fixed, parent base_link, child camera_link, origin xyz=-0.175 0 0.41 rpy=0 0 0

Commit message: added amcl and move_base files for autonomous navigation of robot. Mapping is done but navigation is not working correctly

File: box_robot11/urdf/box_robot11.urdf (robot description, URDF)
Before this commit: robot box_robot11, 8 links, 7 joints
Links:
- link camera_link: geometry collision box size=0.01 0.01 0.35; visual box size=0.05 0.05 0.35
Joints:
- joint joint_sensor_camera: origin xyz=-0.175 0 0.41 rpy=0 0 0 -> xyz=-0.175 0 0.485 rpy=0 0 0
- joint joint_sensor_laser: origin xyz=0.225 0 0.105 rpy=0 0 0 -> xyz=0.155 -0.05 0.025 rpy=1.57075 -1.57075 0; parent base_link -> slider_link

Commit message: Made a new map and tweaked diff_drive parameters to stailize the robot whe working with move_base and amcl. Amcl is working now

File: box_robot11/urdf/box_robot11.urdf (robot description, URDF)
Before this commit: robot box_robot11, 8 links, 7 joints
Links:
- removed link dummy
Joints:
- removed joint dummy_joint
- joint left_joint: axis 0 0 1 -> 0 0 -1
- joint right_joint: axis 0 0 1 -> 0 0 -1
- joint slider_joint: limit lower=-0.3 upper=0 effort=10000 velocity=5.0 -> lower=-0.3 upper=0 effort=10000 velocity=20.0
